Commit message: Changers for me specific setup.

File: fairino3_v6_moveit2_config/config/fairino3_v6_robot.ros2_control.xacro (robot description, xacro)
@@ -1,48 +1,65 @@
 <?xml version="1.0"?>
-<robot xmlns:xacro="http://www.ros.org/wiki/xacro">
-    <xacro:macro name="fairino3_v6_robot_ros2_control" params="name initial_positions_file">
-        <xacro:property name="initial_positions" value="${load_yaml(initial_positions_file)['initial_positions']}"/>
-        <ros2_control name="${name}" type="system">
-            <hardware>
-                <!-- By default, set up controllers for simulation. This won't work on real hardware -->
-                <plugin>mock_components/GenericSystem</plugin>
-            </hardware>
-            <joint name="j1">
-                <command_interface name="position"/>
-                <state_interface name="position">
-                  <param name="initial_value">${initial_positions['j1']}</param>
-                </state_interface>
-            </joint>
-            <joint name="j2">
-                <command_interface name="position"/>
-                <state_interface name="position">
-                  <param name="initial_value">${initial_positions['j2']}</param>
-                </state_interface>
-            </joint>
-            <joint name="j3">
-                <command_interface name="position"/>
-                <state_interface name="position">
-                  <param name="initial_value">${initial_positions['j3']}</param>
-                </state_interface>
-            </joint>
-            <joint name="j4">
-                <command_interface name="position"/>
-                <state_interface name="position">
-                  <param name="initial_value">${initial_positions['j4']}</param>
-                </state_interface>
-            </joint>
-            <joint name="j5">
-                <command_interface name="position"/>
-                <state_interface name="position">
-                  <param name="initial_value">${initial_positions['j5']}</param>
-                </state_interface>
-            </joint>
-            <joint name="j6">
-                <command_interface name="position"/>
-                <state_interface name="position">
-                  <param name="initial_value">${initial_positions['j6']}</param>
-                </state_interface>
-            </joint>
-        </ros2_control>
-    </xacro:macro>
+<robot xmlns:xacro="http://www.ros.org/wiki/xacro" name="fairino3_v6_robot">
+  <xacro:macro name="fairino3_v6_robot_ros2_control" params="name initial_positions_file sim">
+    <xacro:property name="initial_positions" value="${load_yaml(initial_positions_file)['initial_positions']}"/>
+    <webots>
+      <plugin type="webots_ros2_control::Ros2Control"/>
+    </webots>
+    <ros2_control name="${name}" type="system">
+      <hardware>
+        <xacro:if value="${sim}">
+          <plugin>webots_ros2_control::Ros2ControlSystem</plugin>
+        </xacro:if>
+        <xacro:unless value="${sim}">
+          <plugin>fairino_hardware/FairinoHardwareInterface</plugin>
+        </xacro:unless>
+      </hardware>
+      <joint name="j1">
+        <command_interface name="position"/>
+        <state_interface name="position">
+          <param name="initial_value">${initial_positions['j1']}</param>
+        </state_interface>
+        <state_interface name="velocity"/>
+        <state_interface name="effort"/>
+      </joint>
+      <joint name="j2">
+        <command_interface name="position"/>
+        <state_interface name="position">
+          <param name="initial_value">${initial_positions['j2']}</param>
+        </state_interface>
+        <state_interface name="velocity"/>
+        <state_interface name="effort"/>
+      </joint>
+      <joint name="j3">
+        <command_interface name="position"/>
+        <state_interface name="position">
+          <param name="initial_value">${initial_positions['j3']}</param>
+        </state_interface>
+      </joint>
+      <joint name="j4">
+        <command_interface name="position"/>
+        <state_interface name="position">
+          <param name="initial_value">${initial_positions['j4']}</param>
+        </state_interface>
+        <state_interface name="velocity"/>
+        <state_interface name="effort"/>
+      </joint>
+      <joint name="j5">
+        <command_interface name="position"/>
+        <state_interface name="position">
+          <param name="initial_value">${initial_positions['j5']}</param>
+        </state_interface>
+        <state_interface name="velocity"/>
+        <state_interface name="effort"/>
+      </joint>
+      <joint name="j6">
+        <command_interface name="position"/>
+        <state_interface name="position">
+          <param name="initial_value">${initial_positions['j6']}</param>
+        </state_interface>
+        <state_interface name="velocity"/>
+        <state_interface name="effort"/>
+      </joint>
+    </ros2_control>
+  </xacro:macro>
 </robot>

File: fairino3_v6_moveit2_config/config/fairino3_v6_robot.urdf.xacro (robot description, xacro)
@@ -1,4 +1,5 @@
 <?xml version="1.0"?>
 <robot xmlns:xacro="http://www.ros.org/wiki/xacro" name="fairino3_v6_robot">
+    <xacro:arg name="sim" default="true" />
     <xacro:arg name="initial_positions_file" default="initial_positions.yaml" />
     <!-- Import fairino3_v6_robot urdf file -->
@@ -6,4 +7,4 @@
     <!-- Import control_xacro -->
     <xacro:include filename="fairino3_v6_robot.ros2_control.xacro" />
-    <xacro:fairino3_v6_robot_ros2_control name="FakeSystem" initial_positions_file="$(arg initial_positions_file)"/>
+    <xacro:fairino3_v6_robot_ros2_control name="FakeSystem" initial_positions_file="$(arg initial_positions_file)" sim="$(arg sim)"/>
 </robot>
