Commit message: Added end effector and intitial positions.

File: fairino_description/urdf/fairino3_v6.urdf (robot description, URDF)
Before this commit: robot fairino3_v6_robot, 7 links, 6 joints
Links:
- added link end_effector
Joints:
- added joint eef: type fixed, parent wrist3_link, child end_effector, origin xyz=0 0 0.100 rpy=0 0 0

Commit message: More edits.

File: fairino_description/urdf/fairino3_v6.urdf (robot description, URDF)
Before this commit: robot fairino3_v6_robot, 8 links, 7 joints
Joints:
- joint eef: origin xyz=0 0 0.100 rpy=0 0 0 -> xyz=0 0 0.169 rpy=0 0 0

Commit message: Modifed end effector distance.

File: fairino_description/urdf/fairino3_v6.urdf (robot description, URDF)
Before this commit: robot fairino3_v6_robot, 8 links, 7 joints
Joints:
- joint eef: origin xyz=0 0 0.169 rpy=0 0 0 -> xyz=0 0 0.164 rpy=0 0 0

Commit message: Changed end effector distance again.

File: fairino_description/urdf/fairino3_v6.urdf (robot description, URDF)
Before this commit: robot fairino3_v6_robot, 8 links, 7 joints
Joints:
- joint eef: origin xyz=0 0 0.164 rpy=0 0 0 -> xyz=0 0 0.108 rpy=0 0 0
